File: eSim_Project_Files/four_bit_async_counter_Syed_Imaduddin/four_bit_async_counter_Syed_Imaduddin.sch (KiCad schematic (older format))
At the start: 31 parts, among them U1 plot_v1, U10 plot_v1, U11 plot_v1, U12 adc_bridge_3, U13 dac_bridge_4, U14 plot_v1, U2 plot_v1, U3 plot_v1, U4 tff, U5 tff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

Commit message: Everything is updated
Parts:
- removed U4, U5, U6, U9: tff, symbol tff
- added U4, U5, U6, U9: imad_tff, symbol imad_tff
Connections:
- net at U12.4 (OUT1): now also U4.1 (clk0)
- net at U12.5 (OUT2): now also U4.2 (rstn0), U5.2 (rstn0), U6.2 (rstn0), U9.2 (rstn0)
- net at U12.6 (OUT3): now also U4.3 (t0), U5.3 (t0), U6.3 (t0), U9.3 (t0)
- net at U13.1 (IN1): now also U4.4 (q0), U5.1 (clk0)
- net at U13.2 (IN2): now also U5.4 (q0), U6.1 (clk0)
- net at U13.3 (IN3): now also U6.4 (q0), U9.1 (clk0)
- net at U13.4 (IN4): now also U9.4 (q0)
Changed lines of the file:
@@
 LIBS:eSim_SKY130
 LIBS:eSim_SKY130_Subckts
+LIBS:four_bit_async_counter_Syed_Imaduddin-cache
 EELAYER 25 0
 EELAYER END
@@
 in
 $Comp
-L GND #PWR01
+L GND #PWR9
 U 1 1 633C337A
 P 5350 2750
-F 0 "#PWR01" H 5350 2500 50  0001 C CNN
+F 0 "#PWR9" H 5350 2500 50  0001 C CNN
 F 1 "GND" H 5350 2600 50  0000 C CNN
 F 2 "" H 5350 2750 50  0001 C CNN
 F 3 "" H 5350 2750 50  0001 C CNN
 	1    5350 2750
-	1    0    0    -1
-$EndComp
-$Comp
-L tff U4
-U 1 1 633D2ABD
-P 1500 7100
-F 0 "U4" H 4350 8900 60  0000 C CNN
-F 1 "tff" H 4350 9100 60  0000 C CNN
-F 2 "" H 4350 9050 60  0000 C CNN
-F 3 "" H 4350 9050 60  0000 C CNN
-	1    1500 7100
-	1    0    0    -1
-$EndComp
-$Comp
-L tff U5
-U 1 1 633D2D39
-P 3350 7100
-F 0 "U5" H 6200 8900 60  0000 C CNN
-F 1 "tff" H 6200 9100 60  0000 C CNN
-F 2 "" H 6200 9050 60  0000 C CNN
-F 3 "" H 6200 9050 60  0000 C CNN
-	1    3350 7100
-	1    0    0    -1
-$EndComp
-$Comp
-L tff U6
-U 1 1 633D2E56
-P 5150 7100
-F 0 "U6" H 8000 8900 60  0000 C CNN
-F 1 "tff" H 8000 9100 60  0000 C CNN
-F 2 "" H 8000 9050 60  0000 C CNN
-F 3 "" H 8000 9050 60  0000 C CNN
-	1    5150 7100
-	1    0    0    -1
-$EndComp
-$Comp
-L tff U9
-U 1 1 633D2F8A
-P 7000 7100
-F 0 "U9" H 9850 8900 60  0000 C CNN
-F 1 "tff" H 9850 9100 60  0000 C CNN
-F 2 "" H 9850 9050 60  0000 C CNN
-F 3 "" H 9850 9050 60  0000 C CNN
-	1    7000 7100
 	1    0    0    -1
 $EndComp
@@
 $EndComp
 $Comp
-L GND #PWR02
+L GND #PWR10
 U 1 1 633DB644
 P 8700 3800
-F 0 "#PWR02" H 8700 3550 50  0001 C CNN
+F 0 "#PWR10" H 8700 3550 50  0001 C CNN
 F 1 "GND" H 8700 3650 50  0000 C CNN
 F 2 "" H 8700 3800 50  0001 C CNN
@@
 $EndComp
 $Comp
-L GND #PWR03
+L GND #PWR11
 U 1 1 633DB694
 P 9450 3800
-F 0 "#PWR03" H 9450 3550 50  0001 C CNN
+F 0 "#PWR11" H 9450 3550 50  0001 C CNN
 F 1 "GND" H 9450 3650 50  0000 C CNN
 F 2 "" H 9450 3800 50  0001 C CNN
@@
 $EndComp
 $Comp
-L GND #PWR04
+L GND #PWR12
 U 1 1 633DB6E4
 P 10150 3800
-F 0 "#PWR04" H 10150 3550 50  0001 C CNN
+F 0 "#PWR12" H 10150 3550 50  0001 C CNN
 F 1 "GND" H 10150 3650 50  0000 C CNN
 F 2 "" H 10150 3800 50  0001 C CNN
@@
 $EndComp
 $Comp
-L GND #PWR05
+L GND #PWR13
 U 1 1 633DB734
 P 10800 3800
-F 0 "#PWR05" H 10800 3550 50  0001 C CNN
+F 0 "#PWR13" H 10800 3550 50  0001 C CNN
 F 1 "GND" H 10800 3650 50  0000 C CNN
 F 2 "" H 10800 3800 50  0001 C CNN
@@
 $EndComp
 $Comp
-L GND #PWR06
+L GND #PWR3
 U 1 1 634072D4
 P 1750 3500
-F 0 "#PWR06" H 1750 3250 50  0001 C CNN
+F 0 "#PWR3" H 1750 3250 50  0001 C CNN
 F 1 "GND" H 1750 3350 50  0000 C CNN
 F 2 "" H 1750 3500 50  0001 C CNN
@@
 $EndComp
 $Comp
-L GND #PWR07
+L GND #PWR5
 U 1 1 63407DAA
 P 2900 3500
-F 0 "#PWR07" H 2900 3250 50  0001 C CNN
+F 0 "#PWR5" H 2900 3250 50  0001 C CNN
 F 1 "GND" H 2900 3350 50  0000 C CNN
 F 2 "" H 2900 3500 50  0001 C CNN
@@
 $EndComp
 $Comp
-L GND #PWR08
+L GND #PWR7
 U 1 1 63407E63
 P 4000 3500
-F 0 "#PWR08" H 4000 3250 50  0001 C CNN
+F 0 "#PWR7" H 4000 3250 50  0001 C CNN
 F 1 "GND" H 4000 3350 50  0000 C CNN
 F 2 "" H 4000 3500 50  0001 C CNN
@@
 $EndComp
 $Comp
-L GND #PWR09
+L GND #PWR8
 U 1 1 634087A5
 P 4300 3450
-F 0 "#PWR09" H 4300 3200 50  0001 C CNN
+F 0 "#PWR8" H 4300 3200 50  0001 C CNN
 F 1 "GND" H 4300 3300 50  0000 C CNN
 F 2 "" H 4300 3450 50  0001 C CNN
@@
 $EndComp
 $Comp
-L GND #PWR010
+L GND #PWR6
 U 1 1 634087F7
 P 3200 3450
-F 0 "#PWR010" H 3200 3200 50  0001 C CNN
+F 0 "#PWR6" H 3200 3200 50  0001 C CNN
 F 1 "GND" H 3200 3300 50  0000 C CNN
 F 2 "" H 3200 3450 50  0001 C CNN
@@
 $EndComp
 $Comp
-L GND #PWR011
+L GND #PWR4
 U 1 1 63408849
 P 2100 3450
-F 0 "#PWR011" H 2100 3200 50  0001 C CNN
+F 0 "#PWR4" H 2100 3200 50  0001 C CNN
 F 1 "GND" H 2100 3300 50  0000 C CNN
 F 2 "" H 2100 3450 50  0001 C CNN
@@
 $EndComp
 $Comp
-L GND #PWR012
+L GND #PWR2
 U 1 1 634099A8
 P 1500 6850
-F 0 "#PWR012" H 1500 6600 50  0001 C CNN
+F 0 "#PWR2" H 1500 6600 50  0001 C CNN
 F 1 "GND" H 1500 6700 50  0000 C CNN
 F 2 "" H 1500 6850 50  0001 C CNN
@@
 $EndComp
 $Comp
-L GND #PWR013
+L GND #PWR1
 U 1 1 634099FA
 P 850 6750
-F 0 "#PWR013" H 850 6500 50  0001 C CNN
+F 0 "#PWR1" H 850 6500 50  0001 C CNN
 F 1 "GND" H 850 6600 50  0000 C CNN
 F 2 "" H 850 6750 50  0001 C CNN
@@
 	1900 1950 1900 1500
 Connection ~ 1900 1500
+$Comp
+L imad_tff U4
+U 1 1 63410D56
+P 1500 7100
+F 0 "U4" H 4350 8900 60  0000 C CNN
+F 1 "imad_tff" H 4350 9100 60  0000 C CNN
+F 2 "" H 4350 9050 60  0000 C CNN
+F 3 "" H 4350 9050 60  0000 C CNN
+	1    1500 7100
+	1    0    0    -1
+$EndComp
+$Comp
+L imad_tff U5
+U 1 1 634114E2
+P 3350 7100
+F 0 "U5" H 6200 8900 60  0000 C CNN
+F 1 "imad_tff" H 6200 9100 60  0000 C CNN
+F 2 "" H 6200 9050 60  0000 C CNN
+F 3 "" H 6200 9050 60  0000 C CNN
+	1    3350 7100
+	1    0    0    -1
+$EndComp
+$Comp
+L imad_tff U6
+U 1 1 63411B63
+P 5150 7100
+F 0 "U6" H 8000 8900 60  0000 C CNN
+F 1 "imad_tff" H 8000 9100 60  0000 C CNN
+F 2 "" H 8000 9050 60  0000 C CNN
+F 3 "" H 8000 9050 60  0000 C CNN
+	1    5150 7100
+	1    0    0    -1
+$EndComp
+$Comp
+L imad_tff U9
+U 1 1 63412358
+P 7000 7100
+F 0 "U9" H 9850 8900 60  0000 C CNN
+F 1 "imad_tff" H 9850 9100 60  0000 C CNN
+F 2 "" H 9850 9050 60  0000 C CNN
+F 3 "" H 9850 9050 60  0000 C CNN
+	1    7000 7100
+	1    0    0    -1
+$EndComp
 $EndSCHEMATC
